Commit message: Day 77 add ros2_control foundation

File: ros2_ws/src/cpp_robotics_sim_ros/xacro/diffbot.xacro (robot description, xacro)
@@ -177,3 +177,29 @@
     <origin xyz="${caster_x} ${caster_y} ${caster_z}" rpy="0 0 0"/>
   </joint>
+	<ros2_control name="DiffBotSystem" type="system">
+		<hardware>
+			<plugin>gz_ros2_control/GazeboSimSystem</plugin>
+		</hardware>
+		<joint name="left_wheel_joint">
+			<command_interface name="velocity">
+				<param name="min">-10.0</param>
+				<param name="max">10.0</param>
+			</command_interface>
+			<state_interface name="position"/>
+			<state_interface name="velocity"/>
+		</joint>
+		<joint name="right_wheel_joint">
+			<command_interface name="velocity">
+				<param name="min">-10.0</param>
+				<param name="max">10.0</param>
+			</command_interface>
+			<state_interface name="position"/>
+			<state_interface name="velocity"/>
+		</joint>
+	</ros2_control>
+	<gazebo>
+		<plugin filename="gz_ros2_control-system" name="gz_ros2_control::GazeboSimROS2ControlPlugin">
+			<parameters>$(find cpp_robotics_sim_ros)/config/ros2_control.yaml</parameters>
+		</plugin>
+	</gazebo>
 </robot>

Commit message: Day 79 add simulated lidar sensor

File: ros2_ws/src/cpp_robotics_sim_ros/xacro/diffbot.xacro (robot description, xacro)
@@ -157,4 +157,33 @@
       radius="${caster_radius}"/>
   </link>
+	<link name="lidar_link">
+		<visual>
+			<geometry>
+				<cylinder radius="0.04" length="0.04"/>
+			</geometry>
+			<origin xyz="0 0 0" rpy="0 0 0"/>
+			<material name="blue">
+				<color rgba="0.0 0.2 1.0 1.0"/>
+			</material>
+		</visual>
+		<collision>
+			<geometry>
+				<cylinder radius="0.04" length="0.04"/>
+			</geometry>
+			<origin xyz="0 0 0" rpy="0 0 0"/>
+		</collision>
+		<inertial>
+			<mass value="0.05"/>
+			<origin xyz="0 0 0" rpy="0 0 0"/>
+			<inertia ixx="0.00005" ixy="0.0" ixz="0.0"
+					 iyy="0.00005" iyz="0.0"
+					 izz="0.00005"/>
+		</inertial>
+	</link>
+	<joint name="lidar_joint" type="fixed">
+		<parent link="base_link"/>
+		<child link="lidar_link"/>
+		<origin xyz="0.15 0 0.18" rpy="0 0 0"/>
+	</joint>
   <!-- ========================= -->
   <!-- Joints                    -->
@@ -198,4 +227,27 @@
 		</joint>
 	</ros2_control>
+	<gazebo reference="lidar_link">
+		<sensor name="diffbot_lidar" type="gpu_lidar">
+			<topic>/scan</topic>
+			<update_rate>10</update_rate>
+			<ray>
+				<scan>
+					<horizontal>
+						<samples>360</samples>
+						<resolution>1</resolution>
+						<min_angle>-3.14159</min_angle>
+						<max_angle>3.14159</max_angle>
+					</horizontal>
+				</scan>
+				<range>
+					<min>0.08</min>
+					<max>8.0</max>
+					<resolution>0.01</resolution>
+				</range>
+			</ray>
+			<always_on>true</always_on>
+			<visualize>true</visualize>
+		</sensor>
+	</gazebo>
 	<gazebo>
 		<plugin filename="gz_ros2_control-system" name="gz_ros2_control::GazeboSimROS2ControlPlugin">
